File: pcb/vyper_f4.kicad_pcb (KiCad board)
At the start: 2 copper layers, 30 x 64 mm, 35 parts, among them J1 J1_usb_service_SH4, J2 J2_esc_SH8, J7 J7_swd_testpads, J8 J8_beeper_pads, T1 PAD_T1, T3 PAD_T3, T6 PAD_T6, U1 U1_mcu_STM32F405RGT6, U2 U2_gyro_ICM42688P, U3 U3_buck_TPS54360, U4 U4_ldo_3v3, U5 U5_gyro_ldo_AP2112K, U6 U6_flash_W25Q128, U7 U7_baro_BMP280, U8 U8_rgb_level_shifter, Y1 Y1_xtal_8MHz

Commit message: Route Vyper FC power gyro bus and clock
Parts:
- U4: moved to B.Cu
- moved Y1 11.2 mm to (4.00, 1.00)
- moved U6 6.67 mm to (-6.50, 9.50)
- moved U3 4.52 mm to (0.00, -17.0)
- moved U4 3.00 mm to (8.50, -18.0)
- moved L1 2.14 mm to (-8.00, -19.7)
- moved U1 2.00 mm to (2.00, 9.50)
Changed lines of the file:
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@@
 		(pad "1" smd roundrect (at 0.000 0.000) (size 2.0 2.0) (layers "F.Cu" "F.Paste" "F.Mask") (roundrect_rratio 0.25))
 	)
-	(gr_rect (start -6.200 3.200) (end 6.200 15.600) (stroke (width 0.05) (type solid)) (fill no) (layer "F.CrtYd"))
-	(gr_rect (start -6.200 3.200) (end 6.200 15.600) (stroke (width 0.12) (type solid)) (fill no) (layer "F.SilkS"))
+	(gr_rect (start -4.200 3.300) (end 8.200 15.700) (stroke (width 0.05) (type solid)) (fill no) (layer "F.CrtYd"))
+	(gr_rect (start -4.200 3.300) (end 8.200 15.700) (stroke (width 0.12) (type solid)) (fill no) (layer "F.SilkS"))
 	(footprint "VYPER:U1_mcu_STM32F405RGT6" (layer "F.Cu")
-		(at 0.000 9.400)
+		(at 2.000 9.500)
 		(attr exclude_from_pos_files)
 		(property "Reference" "U1" (at 0 -2.4 0) (layer "F.SilkS")
@@
 		(pad "1" smd roundrect (at 0.000 0.000) (size 2.0 2.0) (layers "F.Cu" "F.Paste" "F.Mask") (roundrect_rratio 0.25))
 	)
-	(gr_rect (start 7.400 9.250) (end 10.600 12.750) (stroke (width 0.05) (type solid)) (fill no) (layer "B.CrtYd"))
-	(gr_rect (start 7.400 9.250) (end 10.600 12.750) (stroke (width 0.12) (type solid)) (fill no) (layer "B.SilkS"))
+	(gr_rect (start 1.850 -0.800) (end 6.150 2.800) (stroke (width 0.05) (type solid)) (fill no) (layer "B.CrtYd"))
+	(gr_rect (start 1.850 -0.800) (end 6.150 2.800) (stroke (width 0.12) (type solid)) (fill no) (layer "B.SilkS"))
 	(footprint "VYPER:Y1_xtal_8MHz" (layer "B.Cu")
-		(at 9.000 11.000)
+		(at 4.000 1.000)
 		(attr exclude_from_pos_files)
 		(property "Reference" "Y1" (at 0 -2.4 0) (layer "B.SilkS")
@@
 		(pad "1" smd roundrect (at 0.000 0.000) (size 2.0 2.0) (layers "F.Cu" "F.Paste" "F.Mask") (roundrect_rratio 0.25))
 	)
-	(gr_rect (start -3.250 5.250) (end 3.250 10.750) (stroke (width 0.05) (type solid)) (fill no) (layer "B.CrtYd"))
-	(gr_rect (start -3.250 5.250) (end 3.250 10.750) (stroke (width 0.12) (type solid)) (fill no) (layer "B.SilkS"))
+	(gr_rect (start -11.200 6.550) (end -1.800 12.450) (stroke (width 0.05) (type solid)) (fill no) (layer "B.CrtYd"))
+	(gr_rect (start -11.200 6.550) (end -1.800 12.450) (stroke (width 0.12) (type solid)) (fill no) (layer "B.SilkS"))
 	(footprint "VYPER:U6_flash_W25Q128" (layer "B.Cu")
-		(at 0.000 8.000)
+		(at -6.500 9.500)
 		(attr exclude_from_pos_files)
 		(property "Reference" "U6" (at 0 -2.4 0) (layer "B.SilkS")
@@
 		(pad "1" smd roundrect (at 0.000 0.000) (size 2.0 2.0) (layers "B.Cu" "B.Paste" "B.Mask") (roundrect_rratio 0.25))
 	)
-	(gr_rect (start -8.600 -23.300) (end -4.000 -18.700) (stroke (width 0.05) (type solid)) (fill no) (layer "F.CrtYd"))
-	(gr_rect (start -8.600 -23.300) (end -4.000 -18.700) (stroke (width 0.12) (type solid)) (fill no) (layer "F.SilkS"))
+	(gr_rect (start -12.200 -23.450) (end -3.800 -15.950) (stroke (width 0.05) (type solid)) (fill no) (layer "F.CrtYd"))
+	(gr_rect (start -12.200 -23.450) (end -3.800 -15.950) (stroke (width 0.12) (type solid)) (fill no) (layer "F.SilkS"))
 	(footprint "VYPER:L1_buck_inductor" (layer "F.Cu")
-		(at -6.300 -21.000)
+		(at -8.000 -19.700)
 		(attr exclude_from_pos_files)
 		(property "Reference" "L1" (at 0 -2.4 0) (layer "F.SilkS")
@@
 		(pad "1" smd roundrect (at 0.000 0.000) (size 2.0 2.0) (layers "F.Cu" "F.Paste" "F.Mask") (roundrect_rratio 0.25))
 	)
-	(gr_rect (start -1.000 -23.600) (end 5.200 -18.400) (stroke (width 0.05) (type solid)) (fill no) (layer "F.CrtYd"))
-	(gr_rect (start -1.000 -23.600) (end 5.200 -18.400) (stroke (width 0.12) (type solid)) (fill no) (layer "F.SilkS"))
+	(gr_rect (start -2.800 -20.800) (end 2.800 -13.200) (stroke (width 0.05) (type solid)) (fill no) (layer "F.CrtYd"))
+	(gr_rect (start -2.800 -20.800) (end 2.800 -13.200) (stroke (width 0.12) (type solid)) (fill no) (layer "F.SilkS"))
 	(footprint "VYPER:U3_buck_TPS54360" (layer "F.Cu")
-		(at 2.100 -21.000)
+		(at 0.000 -17.000)
 		(attr exclude_from_pos_files)
 		(property "Reference" "U3" (at 0 -2.4 0) (layer "F.SilkS")
@@
 		(pad "1" smd roundrect (at 0.000 0.000) (size 2.0 2.0) (layers "F.Cu" "F.Paste" "F.Mask") (roundrect_rratio 0.25))
 	)
-	(gr_rect (start 6.700 -22.600) (end 10.100 -19.400) (stroke (width 0.05) (type solid)) (fill no) (layer "F.CrtYd"))
-	(gr_rect (start 6.700 -22.600) (end 10.100 -19.400) (stroke (width 0.12) (type solid)) (fill no) (layer "F.SilkS"))
-	(footprint "VYPER:U4_ldo_3v3" (layer "F.Cu")
-		(at 8.400 -21.000)
+	(gr_rect (start 6.400 -19.750) (end 10.600 -16.250) (stroke (width 0.05) (type solid)) (fill no) (layer "B.CrtYd"))
+	(gr_rect (start 6.400 -19.750) (end 10.600 -16.250) (stroke (width 0.12) (type solid)) (fill no) (layer "B.SilkS"))
+	(footprint "VYPER:U4_ldo_3v3" (layer "B.Cu")
+		(at 8.500 -18.000)
 		(attr exclude_from_pos_files)
-		(property "Reference" "U4" (at 0 -2.4 0) (layer "F.SilkS")
-			(effects (font (size 0.8 0.8) (thickness 0.12)))
+		(property "Reference" "U4" (at 0 -2.4 0) (layer "B.SilkS")
+			(effects (font (size 0.8 0.8) (thickness 0.12)) (justify mirror))
 		)
-		(property "Value" "U4_ldo_3v3" (at 0 2.4 0) (layer "F.SilkS")
+		(property "Value" "U4_ldo_3v3" (at 0 2.4 0) (layer "B.SilkS")
 			(effects (font (size 0.5 0.5) (thickness 0.08)) (hide yes))
 		)
-		(pad "1" smd roundrect (at 0.000 0.000) (size 2.0 2.0) (layers "F.Cu" "F.Paste" "F.Mask") (roundrect_rratio 0.25))
+		(pad "1" smd roundrect (at 0.000 0.000) (size 2.0 2.0) (layers "B.Cu" "B.Paste" "B.Mask") (roundrect_rratio 0.25))
 	)
 	(gr_rect (start -3.500 26.200) (end 3.500 30.800) (stroke (width 0.05) (type solid)) (fill no) (layer "B.CrtYd"))

Commit message: Route STM32 VCAP regulator networks
Parts:
- moved U6 14.5 mm to (8.00, 10.0)
- moved Y1 13.0 mm to (-7.00, 8.00)
- moved U5 2.69 mm to (5.00, -2.00)
Changed lines of the file:
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@@
 		(pad "1" smd roundrect (at 0.000 0.000) (size 2.0 2.0) (layers "F.Cu" "F.Paste" "F.Mask") (roundrect_rratio 0.25))
 	)
-	(gr_rect (start 1.850 -0.800) (end 6.150 2.800) (stroke (width 0.05) (type solid)) (fill no) (layer "B.CrtYd"))
-	(gr_rect (start 1.850 -0.800) (end 6.150 2.800) (stroke (width 0.12) (type solid)) (fill no) (layer "B.SilkS"))
+	(gr_rect (start -9.150 6.200) (end -4.850 9.800) (stroke (width 0.05) (type solid)) (fill no) (layer "B.CrtYd"))
+	(gr_rect (start -9.150 6.200) (end -4.850 9.800) (stroke (width 0.12) (type solid)) (fill no) (layer "B.SilkS"))
 	(footprint "VYPER:Y1_xtal_8MHz" (layer "B.Cu")
-		(at 4.000 1.000)
+		(at -7.000 8.000)
 		(attr exclude_from_pos_files)
 		(property "Reference" "Y1" (at 0 -2.4 0) (layer "B.SilkS")
@@
 		(pad "1" smd roundrect (at 0.000 0.000) (size 2.0 2.0) (layers "B.Cu" "B.Paste" "B.Mask") (roundrect_rratio 0.25))
 	)
-	(gr_rect (start 5.100 -1.600) (end 8.500 1.600) (stroke (width 0.05) (type solid)) (fill no) (layer "F.CrtYd"))
-	(gr_rect (start 5.100 -1.600) (end 8.500 1.600) (stroke (width 0.12) (type solid)) (fill no) (layer "F.SilkS"))
+	(gr_rect (start 3.300 -3.600) (end 6.700 -0.400) (stroke (width 0.05) (type solid)) (fill no) (layer "F.CrtYd"))
+	(gr_rect (start 3.300 -3.600) (end 6.700 -0.400) (stroke (width 0.12) (type solid)) (fill no) (layer "F.SilkS"))
 	(footprint "VYPER:U5_gyro_ldo_AP2112K" (layer "F.Cu")
-		(at 6.800 -0.000)
+		(at 5.000 -2.000)
 		(attr exclude_from_pos_files)
 		(property "Reference" "U5" (at 0 -2.4 0) (layer "F.SilkS")
@@
 		(pad "1" smd roundrect (at 0.000 0.000) (size 2.0 2.0) (layers "F.Cu" "F.Paste" "F.Mask") (roundrect_rratio 0.25))
 	)
-	(gr_rect (start -11.200 6.550) (end -1.800 12.450) (stroke (width 0.05) (type solid)) (fill no) (layer "B.CrtYd"))
-	(gr_rect (start -11.200 6.550) (end -1.800 12.450) (stroke (width 0.12) (type solid)) (fill no) (layer "B.SilkS"))
+	(gr_rect (start 5.050 5.300) (end 10.950 14.700) (stroke (width 0.05) (type solid)) (fill no) (layer "B.CrtYd"))
+	(gr_rect (start 5.050 5.300) (end 10.950 14.700) (stroke (width 0.12) (type solid)) (fill no) (layer "B.SilkS"))
 	(footprint "VYPER:U6_flash_W25Q128" (layer "B.Cu")
-		(at -6.500 9.500)
+		(at 8.000 10.000)
 		(attr exclude_from_pos_files)
 		(property "Reference" "U6" (at 0 -2.4 0) (layer "B.SilkS")
